Commit message: Update gazebo launch file and URDF for trailerbot configuration

File: trailerbot_description/urdf/trailerbot.urdf (robot description, URDF)
Before this commit: robot trailerbot, 12 links, 11 joints
Links:
- link drawbar_link: mass None -> 0.5
- link pivot_marker_link: mass None -> 0.1; geometry collision sphere radius=0.08; visual sphere radius=0.08
Joints:
- joint pivot_marker_drawbar_joint: type revolute -> continuous

Commit message: - urdf updated - rviz config added

File: trailerbot_description/urdf/trailerbot.urdf (robot description, URDF)
Before this commit: robot trailerbot, 12 links, 11 joints
Links:
- link container: mass 20.0 -> 10.0
Joints:
- joint pivot_marker_drawbar_joint: type continuous -> revolute

Commit message: four wheel container added

File: trailerbot_description/urdf/trailerbot.urdf (robot description, URDF)
Before this commit: robot trailerbot, 12 links, 11 joints
Links:
- removed link container_caster_wheel
- removed link container_left_wheel
- removed link container_right_wheel
- added link container_front_left_wheel, mass 0.1; collision cylinder length=0.1 radius=0.1; visual cylinder length=0.1 radius=0.1
- added link container_front_right_wheel, mass 0.1; collision cylinder length=0.1 radius=0.1; visual cylinder length=0.1 radius=0.1
- added link container_rear_left_wheel, mass 0.1; collision cylinder length=0.1 radius=0.1; visual cylinder length=0.1 radius=0.1
- added link container_rear_right_wheel, mass 0.1; collision cylinder length=0.1 radius=0.1; visual cylinder length=0.1 radius=0.1
Joints:
- removed joint container_caster_wheel_joint
- removed joint container_left_wheel_joint
- removed joint container_right_wheel_joint
- added joint container_front_left_wheel_joint: type continuous, parent container, child container_front_left_wheel, origin xyz=1.0 0.5 -0.5 rpy=0 0 0, axis 0 1 0
- added joint container_front_right_wheel_joint: type continuous, parent container, child container_front_right_wheel, origin xyz=1.0 -0.5 -0.5 rpy=0 0 0, axis 0 1 0
- added joint container_rear_left_wheel_joint: type continuous, parent container, child container_rear_left_wheel, origin xyz=-1.0 0.5 -0.5 rpy=0 0 0, axis 0 1 0
- added joint container_rear_right_wheel_joint: type continuous, parent container, child container_rear_right_wheel, origin xyz=-1.0 -0.5 -0.5 rpy=0 0 0, axis 0 1 0
- joint caster_wheel_joint: origin xyz=0.35 0 -0.125 rpy=0 1.571 0 -> xyz=0.35 0 -0.125 rpy=0 0 0

Commit message: height adjusted

File: trailerbot_description/urdf/trailerbot.urdf (robot description, URDF)
Before this commit: robot trailerbot, 13 links, 12 joints
Joints:
- joint container_joint: origin xyz=-1.75 0 0.4 rpy=0 0 0 -> xyz=-1.75 0 0.375 rpy=0 0 0

Commit message: Implement MPC for trailer docking and adjust related components
- Added a new MPC class for trailer docking in reverse_mpc.py, including state and control weight configurations, physical constraints, and cost function adjustments.
- Updated reverse_trailerbot_mpc_node.py to initialize the MPC with modified parameters and handle goal pose updates.
- Enhanced the Pos class in utils.py to include an is_reverse attribute for state management.
- Modified gazebo.launch.py to adjust simulation verbosity settings.
- Updated trailerbot.urdf to change mass properties, wheel joint types, and friction parameters for improved simulation accuracy.

File: trailerbot_description/urdf/trailerbot.urdf (robot description, URDF)
Before this commit: robot trailerbot, 13 links, 12 joints
Links:
- link base_link: mass 10.0 -> 30.0
- link container: mass 10.0 -> 5.0
- link container_front_left_wheel: geometry collision sphere radius=0.1; visual sphere radius=0.1
- link container_front_right_wheel: geometry collision sphere radius=0.1; visual sphere radius=0.1
Joints:
- joint container_front_left_wheel_joint: axis 0 1 0 -> (none); type continuous -> fixed
- joint container_front_right_wheel_joint: axis 0 1 0 -> (none); type continuous -> fixed
